File: tsac_distribution.kicad_sch (KiCad schematic)
At the start: 25 parts, among them J1 Conn_01x23, J2 Conn_01x02, J21 Conn_01x02, J22 Conn_01x02, J23 Conn_01x02, J31 Conn_01x08, J32 Conn_01x02, J33 Conn_01x02, J41 Conn_01x02, J42 Conn_01x02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

Commit message: *: Add layout
Parts:
- removed TP2: TestPoint, TestPoint:TestPoint_Keystone_5000-5004_Miniature, symbol Connector:TestPoint
- added H1, H2, H3, H4: MountingHole_Pad, MountingHole:MountingHole_3.2mm_M3_Pad_Via, symbol Mechanical:MountingHole_Pad
- C1: value ? -> 10n; footprint (none) -> Capacitor_SMD:C_0603_1608Metric
- J1: footprint (none) -> yfs:AMPSEAL-23-776087; DigiKey # (none) -> A107007-ND; Mfr (none) -> TE Connectivity; Mfr # (none) -> 776087-1; Mouser # (none) -> 571-776087-1
- J2, J43, J44: footprint (none) -> yfs:MolexMicrofitPlus1x2; DigiKey # (none) -> 900-2157601032-ND; Mfr (none) -> Molex; Mfr # (none) -> 2157601032; Mouser # (none) -> 538-215760-1032
- J21, J41, J61: footprint (none) -> yfs:MolexMicrofitPlus1x2; DigiKey # (none) -> 900-2157601022-ND; Mfr (none) -> Molex; Mfr # (none) -> 2157601022; Mouser # (none) -> 538-215760-1022
- J22, J23, J32, J33, J42, J62: footprint (none) -> yfs:MolexMicrofitPlus1x2; DigiKey # (none) -> 900-2157601002-ND; Mfr (none) -> Molex; Mfr # (none) -> 2157601002; Mouser # (none) -> 538-215760-1002
- J31: footprint (none) -> yfs:MolexMicrofitPlus1x8; DigiKey # (none) -> 2-1445088-8-ND; Mfr (none) -> TE Connectivity; Mfr # (none) -> 2-1445088-8; Mouser # (none) -> 571-2-1445088-8
- J45: footprint (none) -> yfs:MolexMicrofitPlus1x8; DigiKey # (none) -> 900-2157601008-ND; Mfr (none) -> Molex; Mfr # (none) -> 2157601008; Mouser # (none) -> 538-215760-1008
- J51: footprint (none) -> yfs:MolexMicrofitPlus1x3; DigiKey # (none) -> 900-2157601003-ND; Mfr (none) -> Molex; Mfr # (none) -> 2157601003; Mouser # (none) -> 538-215760-1003
- R1, R2: value 60 -> 62; footprint (none) -> Resistor_SMD:R_1206_3216Metric; DigiKey # (none) -> 541-62UACT-ND; LCSC # (none) -> C2088119; Mfr (none) -> Vishay; Mfr # (none) -> CRCW120662R0JNEAHP; Mouser # (none) -> 71-CRCW120662R0JNEAH
- R3, R4: footprint (none) -> Resistor_SMD:R_0603_1608Metric
- TP1: footprint TestPoint:TestPoint_Keystone_5000-5004_Miniature -> TestPoint:TestPoint_Keystone_5019_Miniature; DigiKey # (none) -> 36-5019CT-ND; LCSC # (none) -> C238131; Mfr (none) -> Keystone Electronics; Mfr # (none) -> 5019; Mouser # (none) -> 534-5019
- renumbered TP3 to TP2, TP4 to TP3
Connections:
- net 12V_BMS: now also J1.3 (Pin_3); no longer J1.21 (Pin_21)
- net 12V_FAN: now also J1.1 (Pin_1); no longer J1.17 (Pin_17)
- net 12V_HV_DET: now also J1.4 (Pin_4); no longer J1.18 (Pin_18)
- net 12V_IMD: now also J1.2 (Pin_2); no longer J1.20 (Pin_20)
- net 12V_PRCHG: now also J1.17 (Pin_17); no longer J1.19 (Pin_19)
- net 5V_TSAL: now also J1.6 (Pin_6); no longer J1.16 (Pin_16)
- net AIR+_ACT: now also J1.7 (Pin_7); no longer J1.5 (Pin_5)
- net AIR+_INT: now also J1.8 (Pin_8); no longer J1.6 (Pin_6)
- net AIR-_ACT: now also J1.15 (Pin_15); no longer J1.7 (Pin_7)
- net AIR-_INT: now also J1.21 (Pin_21); no longer J1.8 (Pin_8)
- net BMS_OK: now also J1.9 (Pin_9); no longer J1.14 (Pin_14)
- net CANH: now also J1.14 (Pin_14); no longer J1.23 (Pin_23)
- net CANL: now also J1.13 (Pin_13); no longer J1.22 (Pin_22)
- net DISCHG: now also J1.12 (Pin_12); no longer J1.11 (Pin_11)
- net GND: now also J1.18 (Pin_18), J1.19 (Pin_19), J1.20 (Pin_20), H1.1, H2.1, H3.1, H4.1; no longer J1.1 (Pin_1), J1.2 (Pin_2), J1.3 (Pin_3)
- net HV_DET: now also J1.5 (Pin_5); no longer J1.4 (Pin_4)
- net IMD_OK: now also J1.10 (Pin_10); no longer J1.13 (Pin_13)
- net IMD_PWM: now also J1.11 (Pin_11); no longer J1.12 (Pin_12)
- net PRCHG_ACT: now also J1.22 (Pin_22); no longer J1.9 (Pin_9)
- net PRCHG_INT: now also J1.23 (Pin_23); no longer J1.10 (Pin_10)
- net SDN_IN: now also J1.16 (Pin_16); no longer J1.15 (Pin_15)
- net IMD_HOOP: now reaches J31.3 (Pin_3), J33.1 (Pin_1), J33.2 (Pin_2)
- net IMD_TSAC: now reaches J31.4 (Pin_4), J32.1 (Pin_1), J32.2 (Pin_2)
Other:
- note added: "Rear Distribution Connector"
- note removed: "Connector to Rear Distribution"
- moved on the sheet: J1
